File: pcb/PIC_DEV_Board.kicad_pcb (KiCad board)
At the start: 4 copper layers, 51 x 32 mm, 31 parts, among them J1 Conn_01x08_Pin, J3 Conn_01x02_Pin, J4 Conn_01x02_Pin, J5 Conn_01x01_Pin, U3 MCP3002, U4 MCP4801, U5 FT230XS

Commit message: layout changes
Parts:
- moved TP1 0.75 mm to (149.2, 110.5)
Routing:
- net Net-(U1-RC0): track 19.3 -> 27.7 mm, vias 0 -> 2
- net Net-(U1-RA2): track 18.8 -> 24.2 mm, vias 0 -> 2
Changed lines of the file:
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@@
 	(footprint "TestPoint:TestPoint_Pad_1.5x1.5mm"
 		(layer "F.Cu")
-		(at 150 110.5 -90)
+		(at 149.25 110.5 -90)
 		(descr "SMD rectangular pad as test Point, square 1.5mm side length")
 		(tags "test point SMD pad rectangle square")
@@
 	)
 	(segment
-		(start 149.964448 100.45)
-		(end 150.36 100.45)
+		(start 157.4325 99.1)
+		(end 157.4325 99.9)
 		(width 0.2)
 		(layer "F.Cu")
@@
 	(segment
 		(start 157.4325 99.1)
-		(end 157.4325 99.9)
+		(end 157.4325 98.0675)
 		(width 0.2)
 		(layer "F.Cu")
@@
 	)
 	(segment
-		(start 149.035 101.379448)
-		(end 149.964448 100.45)
+		(start 149.25 110.5)
+		(end 151.25 110.5)
 		(width 0.2)
 		(layer "F.Cu")
@@
 	)
 	(segment
-		(start 150 110.5)
-		(end 149.035 109.535)
+		(start 157.4325 99.9)
+		(end 156.8825 100.45)
 		(width 0.2)
 		(layer "F.Cu")
@@
 	)
 	(segment
-		(start 149.035 109.535)
-		(end 149.035 101.379448)
+		(start 157.4325 98.0675)
+		(end 158 97.5)
 		(width 0.2)
 		(layer "F.Cu")
@@
 	)
 	(segment
-		(start 157.4325 99.9)
-		(end 156.8825 100.45)
+		(start 156.8825 100.45)
+		(end 150.36 100.45)
 		(width 0.2)
 		(layer "F.Cu")
 		(net 18)
 	)
+	(via
+		(at 158 97.5)
+		(size 0.6)
+		(drill 0.3)
+		(layers "F.Cu" "B.Cu")
+		(net 18)
+	)
+	(via
+		(at 151.25 110.5)
+		(size 0.6)
+		(drill 0.3)
+		(layers "F.Cu" "B.Cu")
+		(net 18)
+	)
 	(segment
-		(start 156.8825 100.45)
-		(end 150.36 100.45)
+		(start 158 97.5)
+		(end 158 103.75)
 		(width 0.2)
-		(layer "F.Cu")
+		(layer "B.Cu")
 		(net 18)
 	)
 	(segment
-		(start 149.964448 99.18)
-		(end 145.5 103.644448)
+		(start 158 103.75)
+		(end 151.25 110.5)
+		(width 0.2)
+		(layer "B.Cu")
+		(net 18)
+	)
+	(segment
+		(start 155 100)
+		(end 154.75 100)
+		(width 0.2)
+		(layer "F.Cu")
+		(net 19)
+	)
+	(segment
+		(start 154.75 100)
+		(end 154.5 99.75)
 		(width 0.2)
 		(layer "F.Cu")
@@
 	)
 	(segment
-		(start 150.36 99.18)
-		(end 149.964448 99.18)
+		(start 145.5 110.5)
+		(end 147.5 110.5)
+		(width 0.2)
+		(layer "F.Cu")
+		(net 19)
+	)
+	(segment
+		(start 155.5275 99.4725)
+		(end 155 100)
 		(width 0.2)
 		(layer "F.Cu")
@@
 	)
 	(segment
-		(start 145.5 103.644448)
-		(end 145.5 110.5)
+		(start 154.9 99.1)
+		(end 155.5275 99.1)
+		(width 0.2)
+		(layer "F.Cu")
+		(net 19)
+	)
+	(segment
+		(start 154.5 99.75)
+		(end 153.5 99.75)
+		(width 0.2)
+		(layer "F.Cu")
+		(net 19)
+	)
+	(segment
+		(start 155.5275 99.1)
+		(end 155.5275 99.4725)
 		(width 0.2)
 		(layer "F.Cu")
@@
 		(net 19)
 	)
+	(via
+		(at 147.5 110.5)
+		(size 0.6)
+		(drill 0.3)
+		(layers "F.Cu" "B.Cu")
+		(net 19)
+	)
+	(via
+		(at 153.5 99.75)
+		(size 0.6)
+		(drill 0.3)
+		(layers "F.Cu" "B.Cu")
+		(net 19)
+	)
+	(segment
+		(start 147.5 110.5)
+		(end 147.5 105)
+		(width 0.2)
+		(layer "B.Cu")
+		(net 19)
+	)
+	(segment
+		(start 152.75 99.75)
+		(end 153.25 99.75)
+		(width 0.2)
+		(layer "B.Cu")
+		(net 19)
+	)
+	(segment
+		(start 147.5 105)
+		(end 152.75 99.75)
+		(width 0.2)
+		(layer "B.Cu")
+		(net 19)
+	)
+	(segment
+		(start 153.25 99.75)
+		(end 153.5 99.75)
+		(width 0.2)
+		(layer "B.Cu")
+		(net 19)
+	)

Commit message: Rev02 final
Routing:
- net Net-(U1-RA2): track 24.2 -> 23.7 mm
Changed lines of the file:
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@@
 			)
 		)
-		(property ki_fp_filters "R_*")
-		(sheetname "Root")
-		(sheetfile "PIC_DEV_Board.kicad_sch")
 		(attr smd)
 		(fp_line
@@
 			(size 1.025 1.4)
 			(layers "F.Cu" "F.Paste" "F.Mask")
-			(roundrect_rratio 0.243902)
+			(roundrect_rratio 0.243902439)
 			(net 7 "Earth")
 			(pintype "passive")
@@
 			(size 1.025 1.4)
 			(layers "F.Cu" "F.Paste" "F.Mask")
-			(roundrect_rratio 0.243902)
+			(roundrect_rratio 0.243902439)
 			(net 36 "/VBUS_SENSE")
 			(pintype "passive")
@@
 			)
 		)
-		(property ki_fp_filters "R_*")
-		(sheetname "Root")
-		(sheetfile "PIC_DEV_Board.kicad_sch")
 		(attr smd)
 		(fp_line
@@
 			(size 1.025 1.4)
 			(layers "F.Cu" "F.Paste" "F.Mask")
-			(roundrect_rratio 0.243902)
+			(roundrect_rratio 0.243902439)
 			(net 8 "+3V3")
 			(pintype "passive")
@@
 			(size 1.025 1.4)
 			(layers "F.Cu" "F.Paste" "F.Mask")
-			(roundrect_rratio 0.243902)
+			(roundrect_rratio 0.243902439)
 			(net 1 "Net-(D1-A)")
 			(pintype "passive")
@@
 			)
 		)
-		(property ki_fp_filters "R_*")
-		(sheetname "Root")
-		(sheetfile "PIC_DEV_Board.kicad_sch")
 		(attr smd)
 		(fp_line
@@
 			(size 1.025 1.4)
 			(layers "F.Cu" "F.Paste" "F.Mask")
-			(roundrect_rratio 0.243902)
+			(roundrect_rratio 0.243902439)
 			(net 32 "Net-(U1-RA5)")
 			(pintype "passive")
@@
 			(size 1.025 1.4)
 			(layers "F.Cu" "F.Paste" "F.Mask")
-			(roundrect_rratio 0.243902)
+			(roundrect_rratio 0.243902439)
 			(net 31 "Net-(D2-A)")
 			(pintype "passive")
@@
 			)
 		)
-		(property ki_fp_filters "R_*")
-		(sheetname "Root")
-		(sheetfile "PIC_DEV_Board.kicad_sch")
 		(attr smd)
 		(fp_line
@@
 			(size 1.025 1.4)
 			(layers "F.Cu" "F.Paste" "F.Mask")
-			(roundrect_rratio 0.243902)
+			(roundrect_rratio 0.243902439)
 			(net 8 "+3V3")
 			(pintype "passive")
@@
 			(size 1.025 1.4)
 			(layers "F.Cu" "F.Paste" "F.Mask")
-			(roundrect_rratio 0.243902)
+			(roundrect_rratio 0.243902439)
 			(net 25 "/Vpp{slash}RA3{slash}MCLR")
 			(pintype "passive")
@@
 			)
 		)
-		(property ki_fp_filters "R_*")
-		(sheetname "Root")
-		(sheetfile "PIC_DEV_Board.kicad_sch")
 		(attr smd)
 		(fp_line
@@
 			(size 1.025 1.4)
 			(layers "F.Cu" "F.Paste" "F.Mask")
-			(roundrect_rratio 0.243902)
+			(roundrect_rratio 0.243902439)
 			(net 36 "/VBUS_SENSE")
 			(pintype "passive")
@@
 			(size 1.025 1.4)
 			(layers "F.Cu" "F.Paste" "F.Mask")
-			(roundrect_rratio 0.243902)
+			(roundrect_rratio 0.243902439)
 			(net 35 "Net-(U6-VCC)")
 			(pintype "passive")
@@
 	)
 	(segment
-		(start 154.75 100)
-		(end 154.5 99.75)
+		(start 155.35 99.1)
+		(end 155.27 99.18)
 		(width 0.2)
 		(layer "F.Cu")
@@
 	)
 	(segment
-		(start 155.5275 99.1)
-		(end 150.44 99.1)
+		(start 154.75 100)
+		(end 154.5 99.75)
 		(width 0.2)
 		(layer "F.Cu")
@@
 	)
 	(segment
-		(start 154.9 99.1)
-		(end 155.5275 99.1)
+		(start 155.27 99.18)
+		(end 150.36 99.18)
 		(width 0.2)
 		(layer "F.Cu")
@@
 		(width 0.2)
 		(layer "F.Cu")
+		(net 19)
+	)
+	(segment
+		(start 155.5275 99.1)
+		(end 155.35 99.1)
+		(width 0.2)
+		(layer "F.Cu")
